File: hardware/fbri_flight.sch (EAGLE design)
At the start: 36 parts, among them U1 SAM_D20E, U2 SI4060, U3 MAX1947, U4 ANTENOVA_GPS_M10382, U5 S25FS-S

Commit message: Started work on development hardware
Parts:
- C1: value 100nF -> 15pF
- C12: value 100pF -> 100nF
- C14: value 100nF -> 100pF
- R2, R3, R4: value 1kΩ -> 100Ω
- renumbered JTAG2 to JTAG1, U$45 to J1
Connections:
- net 1.2V: now also C14.P$1; no longer C12.P$1
- net 1.8V: now also C12.P$1; no longer C14.P$1
Other:
- note added: "Datasheet suggests both 18pF and 22pF"
- note added: "Flight"
- moved on the sheet: C12, C14
Changed lines of the file:
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@@
 <part name="U$4" library="microbuilder_v3" deviceset="1.8V" device=""/>
 <part name="U$5" library="microbuilder_v3" deviceset="1.8V" device=""/>
-<part name="C1" library="microbuilder_v3" deviceset="CAP_CERAMIC" device="_0402" value="100nF"/>
+<part name="C1" library="microbuilder_v3" deviceset="CAP_CERAMIC" device="_0402" value="15pF"/>
 <part name="U$7" library="microbuilder_v3" deviceset="1.8V" device=""/>
 <part name="C2" library="microbuilder_v3" deviceset="CAP_CERAMIC" device="_0402" value="100nF"/>
@@
 <part name="U$36" library="microbuilder_v3" deviceset="GND" device=""/>
 <part name="U$37" library="microbuilder_v3" deviceset="1.8V" device=""/>
-<part name="R2" library="microbuilder_v3" deviceset="RESISTOR" device="_0402" value="1kΩ"/>
+<part name="R2" library="microbuilder_v3" deviceset="RESISTOR" device="_0402" value="100Ω"/>
 <part name="U5" library="fbri" deviceset="S25FS-S" device=""/>
 <part name="U$39" library="microbuilder_v3" deviceset="GND" device=""/>
 <part name="U$40" library="microbuilder_v3" deviceset="1.8V" device=""/>
-<part name="JTAG2" library="microbuilder_v3" deviceset="JTAG-CORTEXM3" device="SMT"/>
-<part name="R3" library="microbuilder_v3" deviceset="RESISTOR" device="_0402" value="1kΩ"/>
-<part name="R4" library="microbuilder_v3" deviceset="RESISTOR" device="_0402" value="1kΩ"/>
+<part name="JTAG1" library="microbuilder_v3" deviceset="JTAG-CORTEXM3" device="SMT"/>
+<part name="R3" library="microbuilder_v3" deviceset="RESISTOR" device="_0402" value="100Ω"/>
+<part name="R4" library="microbuilder_v3" deviceset="RESISTOR" device="_0402" value="100Ω"/>
 <part name="U$41" library="microbuilder_v3" deviceset="1.8V" device=""/>
 <part name="L2" library="microbuilder_v3" deviceset="INDUCTOR" device="_0402" value="220nH"/>
@@
 <part name="C11" library="microbuilder_v3" deviceset="CAP_CERAMIC" device="_0402" value="100nF"/>
 <part name="U$50" library="microbuilder_v3" deviceset="GND" device=""/>
-<part name="C12" library="microbuilder_v3" deviceset="CAP_CERAMIC" device="_0402" value="100pF"/>
+<part name="C14" library="microbuilder_v3" deviceset="CAP_CERAMIC" device="_0402" value="100pF"/>
 <part name="U$51" library="microbuilder_v3" deviceset="GND" device=""/>
 <part name="C13" library="microbuilder_v3" deviceset="CAP_CERAMIC" device="_0402" value="100pF"/>
 <part name="U$52" library="microbuilder_v3" deviceset="GND" device=""/>
-<part name="C14" library="microbuilder_v3" deviceset="CAP_CERAMIC" device="_0402" value="100nF"/>
+<part name="C12" library="microbuilder_v3" deviceset="CAP_CERAMIC" device="_0402" value="100nF"/>
 <part name="C15" library="microbuilder_v3" deviceset="CAP_CERAMIC" device="_0402" value="100pF"/>
 <part name="C16" library="microbuilder_v3" deviceset="CAP_CERAMIC" device="_0402" value="100pF"/>
@@
 <part name="C18" library="microbuilder_v3" deviceset="CAP_CERAMIC" device="_0402" value="15pF"/>
 <part name="U$58" library="microbuilder_v3" deviceset="GND" device=""/>
-<part name="U$45" library="fbri" deviceset="AAA_HOLDER" device=""/>
+<part name="J1" library="fbri" deviceset="AAA_HOLDER" device=""/>
 <part name="U$46" library="microbuilder_v3" deviceset="GND" device=""/>
 <part name="U$47" library="microbuilder_v3" deviceset="1.2V" device=""/>
@@
 <text x="10.16" y="91.44" size="6.4516" layer="97" font="vector" ratio="11">CPU + Mem + Power</text>
 <text x="266.7" y="149.86" size="6.4516" layer="97" font="vector" ratio="11">Comms</text>
+<text x="403.86" y="25.4" size="6.4516" layer="94" font="vector" ratio="11">Flight</text>
+<text x="149.86" y="25.4" size="6.4516" layer="94" font="vector" ratio="11">Flight</text>
+<text x="281.94" y="58.928" size="1.27" layer="97" font="vector" ratio="11" distance="100">Datasheet suggests
+both 18pF and 22pF</text>
 </plain>
 <instances>
@@
 <instance part="U$32" gate="G$1" x="104.14" y="66.04"/>
 <instance part="U$33" gate="G$1" x="30.48" y="66.04"/>
-<instance part="U$34" gate="G$1" x="332.74" y="81.28" rot="MR0"/>
-<instance part="U$35" gate="G$1" x="335.28" y="81.28" rot="MR0"/>
+<instance part="U$34" gate="G$1" x="332.74" y="86.36" rot="MR0"/>
+<instance part="U$35" gate="G$1" x="335.28" y="86.36" rot="MR0"/>
 <instance part="U$36" gate="G$1" x="340.36" y="78.74"/>
-<instance part="U$37" gate="G$1" x="345.44" y="81.28" rot="MR0"/>
+<instance part="U$37" gate="G$1" x="345.44" y="86.36" rot="MR0"/>
 <instance part="R2" gate="G$1" x="314.96" y="43.18"/>
 <instance part="U5" gate="G$1" x="198.12" y="58.42"/>
 <instance part="U$39" gate="G$1" x="170.18" y="45.72"/>
 <instance part="U$40" gate="G$1" x="170.18" y="71.12" rot="MR0"/>
-<instance part="JTAG2" gate="G$1" x="48.26" y="149.86"/>
+<instance part="JTAG1" gate="G$1" x="48.26" y="149.86"/>
 <instance part="R3" gate="G$1" x="375.92" y="63.5"/>
 <instance part="R4" gate="G$1" x="381" y="60.96"/>
@@
 <instance part="C11" gate="G$1" x="340.36" y="152.4"/>
 <instance part="U$50" gate="G$1" x="340.36" y="147.32"/>
-<instance part="C12" gate="G$1" x="114.3" y="38.1"/>
+<instance part="C14" gate="G$1" x="114.3" y="38.1"/>
 <instance part="U$51" gate="G$1" x="114.3" y="30.48"/>
 <instance part="C13" gate="G$1" x="307.34" y="35.56"/>
 <instance part="U$52" gate="G$1" x="307.34" y="27.94"/>
-<instance part="C14" gate="G$1" x="170.18" y="58.42"/>
+<instance part="C12" gate="G$1" x="170.18" y="58.42"/>
 <instance part="C15" gate="G$1" x="373.38" y="53.34"/>
 <instance part="C16" gate="G$1" x="398.78" y="53.34"/>
@@
 <instance part="C18" gate="G$1" x="320.04" y="152.4"/>
 <instance part="U$58" gate="G$1" x="320.04" y="147.32"/>
-<instance part="U$45" gate="G$1" x="17.78" y="45.72" rot="R270"/>
+<instance part="J1" gate="G$1" x="17.78" y="45.72" rot="R270"/>
 <instance part="U$46" gate="G$1" x="17.78" y="30.48"/>
 <instance part="U$47" gate="G$1" x="17.78" y="66.04"/>
@@
 <pinref part="U$6" gate="G$1" pin="GND"/>
 <junction x="35.56" y="154.94"/>
-<pinref part="JTAG2" gate="G$1" pin="3"/>
-<pinref part="JTAG2" gate="G$1" pin="5"/>
+<pinref part="JTAG1" gate="G$1" pin="3"/>
+<pinref part="JTAG1" gate="G$1" pin="5"/>
 </segment>
 <segment>
@@
 <wire x1="177.8" y1="50.8" x2="170.18" y2="50.8" width="0.1524" layer="91"/>
 <junction x="170.18" y="50.8"/>
-<pinref part="C14" gate="G$1" pin="P$2"/>
+<pinref part="C12" gate="G$1" pin="P$2"/>
 <wire x1="170.18" y1="53.34" x2="170.18" y2="55.88" width="0.1524" layer="91"/>
 <junction x="170.18" y="53.34"/>
@@
 </segment>
 <segment>
-<pinref part="C12" gate="G$1" pin="P$2"/>
+<pinref part="C14" gate="G$1" pin="P$2"/>
 <pinref part="U$51" gate="G$1" pin="GND"/>
 <wire x1="114.3" y1="33.02" x2="114.3" y2="35.56" width="0.1524" layer="91"/>
@@
 <segment>
 <pinref part="U$46" gate="G$1" pin="GND"/>
-<pinref part="U$45" gate="G$1" pin="-"/>
+<pinref part="J1" gate="G$1" pin="-"/>
 <wire x1="17.78" y1="33.02" x2="17.78" y2="41.91" width="0.1524" layer="91"/>
 </segment>
@@
 <pinref part="U1" gate="G$1" pin="PA31/SWDIO"/>
 <wire x1="101.6" y1="137.16" x2="111.76" y2="137.16" width="0.1524" layer="91"/>
-<pinref part="JTAG2" gate="G$1" pin="2"/>
+<pinref part="JTAG1" gate="G$1" pin="2"/>
 </segment>
 </net>
@@
 <wire x1="111.76" y1="139.7" x2="104.14" y2="139.7" width="0.1524" layer="91"/>
 <wire x1="104.14" y1="139.7" x2="104.14" y2="157.48" width="0.1524" layer="91"/>
-<pinref part="JTAG2" gate="G$1" pin="4"/>
+<pinref part="JTAG1" gate="G$1" pin="4"/>
 </segment>
 </net>
@@
 <label x="78.74" y="149.86" size="1.778" layer="95" rot="MR0"/>
 <pinref part="U1" gate="G$1" pin="RESETN"/>
-<pinref part="JTAG2" gate="G$1" pin="10"/>
+<pinref part="JTAG1" gate="G$1" pin="10"/>
 </segment>
 <segment>
@@
 <wire x1="35.56" y1="160.02" x2="38.1" y2="160.02" width="0.1524" layer="91"/>
 <pinref part="U$4" gate="G$1" pin="1.8V"/>
-<pinref part="JTAG2" gate="G$1" pin="1"/>
+<pinref part="JTAG1" gate="G$1" pin="1"/>
 </segment>
 <segment>
@@
 <pinref part="U4" gate="G$1" pin="VCC"/>
 <pinref part="U$34" gate="G$1" pin="1.8V"/>
-<wire x1="332.74" y1="81.28" x2="332.74" y2="78.74" width="0.1524" layer="91"/>
+<wire x1="332.74" y1="81.28" x2="332.74" y2="83.82" width="0.1524" layer="91"/>
 </segment>
 <segment>
 <pinref part="U4" gate="G$1" pin="VIO"/>
 <pinref part="U$35" gate="G$1" pin="1.8V"/>
-<wire x1="335.28" y1="81.28" x2="335.28" y2="78.74" width="0.1524" layer="91"/>
+<wire x1="335.28" y1="81.28" x2="335.28" y2="83.82" width="0.1524" layer="91"/>
 </segment>
 <segment>
 <pinref part="U4" gate="G$1" pin="VDD_RF"/>
 <pinref part="U$37" gate="G$1" pin="1.8V"/>
-<wire x1="345.44" y1="81.28" x2="345.44" y2="78.74" width="0.1524" layer="91"/>
+<wire x1="345.44" y1="81.28" x2="345.44" y2="83.82" width="0.1524" layer="91"/>
 </segment>
 <segment>
@@
 <wire x1="177.8" y1="66.04" x2="170.18" y2="66.04" width="0.1524" layer="91"/>
 <wire x1="170.18" y1="66.04" x2="170.18" y2="68.58" width="0.1524" layer="91"/>
-<pinref part="C14" gate="G$1" pin="P$1"/>
+<pinref part="C12" gate="G$1" pin="P$1"/>
 <wire x1="170.18" y1="63.5" x2="170.18" y2="66.04" width="0.1524" layer="91"/>
 <junction x="170.18" y="66.04"/>
@@
 <junction x="104.14" y="55.88"/>
 <junction x="104.14" y="45.72"/>
-<pinref part="C12" gate="G$1" pin="P$1"/>
+<pinref part="C14" gate="G$1" pin="P$1"/>
 <wire x1="104.14" y1="45.72" x2="114.3" y2="45.72" width="0.1524" layer="91"/>
 <wire x1="114.3" y1="45.72" x2="114.3" y2="43.18" width="0.1524" layer="91"/>
@@
 </segment>
 <segment>
-<pinref part="U$45" gate="G$1" pin="+"/>
+<pinref part="J1" gate="G$1" pin="+"/>
 <pinref part="U$47" gate="G$1" pin="1.2V"/>
 <wire x1="17.78" y1="49.53" x2="17.78" y2="63.5" width="0.1524" layer="91"/>
@@
 <pinref part="C17" gate="G$1" pin="P$1"/>
 <wire x1="330.2" y1="160.02" x2="330.2" y2="157.48" width="0.1524" layer="91"/>
-</segment>
-</net>
+<junction x="330.2" y="160.02"/>
+<junction x="340.36" y="160.02"/>
+</segment>
+</net>
