File: hardware/hf-breakout/bristol_longshot.sch (EAGLE design)
At the start: 22 parts, among them U1 SAM_D20E

Commit message: HF board done
Parts:
- removed C15, C16: 100nF, microbuilder_v3:CAP_CERAMIC_0402
- removed R8, R9: 10kΩ, microbuilder_v3:RESISTOR_0402
- removed X1: (no value), microbuilder_v3:SMACONNECTOR
- added C10: 100pF, microbuilder_v3:CAP_CERAMIC_0402
- added C11: 1µF, microbuilder_v3:CAP_CERAMIC_0402
- added C4, C5, C6, C7, C8, C9: 100nF, microbuilder_v3:CAP_CERAMIC_0402
- added DD, SS: 0Ω, microbuilder_v3:RESISTOR_0402
- added FB1: (no value), microbuilder_v3:FERRITE_0402
- added IC3: TLV70018DCK, tlv700:TLV700DCK
- added J$1, J$2: SMA_EDGE, SparkFun:SMA_EDGE
- added JP1: (no value), SparkFun:M03LOCK
- added L5: 100nH, microbuilder_v3:INDUCTOR_0402
- added U3: AD8354, fbri:AD8354
- C12: value 100nF -> 1µF
- R4: value 0Ω -> 10kΩ
- R5: value 0Ω -> 15kΩ
- R6: value 15kΩ -> 220Ω
- R7: value 15kΩ -> DNP
- renumbered U$1 to U2, U$23 to U6
Connections:
- removed net !OE: R7.2, R8.1, U2.!OE
- removed net !OE_CTRL: R8.2
- new net 3.3V: C11.P$1, IC3.EN, IC3.IN, JP1.1, JTAG1.1
- new net AMPL_OUT: C5.P$1, L5.1, U3.VOUT
- new net AMPL_VPOS: C10.P$1, C6.P$1, FB1.P$1, L5.2, U3.VPOS
- new net HF: C5.P$2, J$2.SIGNAL
- new net HF_CLK: C4.P$1, U2.CLK3
- new net INPT: C4.P$2, U3.INPT
- new net LED_R: R6.1, U1.PA15
- new net N$1: C12.P$1, IC3.OUT, JP1.3
- net 1.8V: now also C8.P$1, FB1.P$2, JP1.2, R4.2; no longer C15.P$1, JTAG1.1, R9.2
- net CLKIN: now also DD.1; no longer R5.1
- net CLKIN_SMA: now also DD.2, J$1.SIGNAL, R7.2; no longer R5.2, X1.ANT
- net GND: now also C10.P$2, C11.P$2, C6.P$2, C7.P$2, C8.P$2, C9.P$2, IC3.GND, J$1.GND@0, J$1.GND@1, J$1.GND@2, J$1.GND@3, J$2.GND@0, J$2.GND@1, J$2.GND@2, J$2.GND@3, R5.1, SS.2, U2.!OE, U3.COM1, U3.COM1_, U3.COM2, U3.EPAD, U3._COM2; no longer C15.P$2, C16.P$2, R4.2, R6.1, X1.GND1, X1.GND2, X1.GND3, X1.GND4
- net INTR: now also R4.1; no longer R9.1
- net LED: now also R6.2; no longer U1.PA15
- net SCL: now also U1.PA05
- net SDA: now also U1.PA04
- net SSC_DIS: now also R5.2; no longer R6.2
- net TCXO_VDD: now also C7.P$1; no longer C12.P$1
- net VDD_CORE: now also C9.P$1; no longer C16.P$1
- net XB: now also SS.1; no longer R4.1
Other:
- note added: "TLV70018"
- moved on the sheet: C12, D1, JTAG1, R4, R5, R6, R7, U1
