File: hardware/main/bristol_longshot.sch (EAGLE design)
At the start: 42 parts, among them U1 SAM_D20E, U2 SI4060, U4 ADP1607ACPZN-R7, U5 S25FS-S

Commit message: Much layout done for new frontpanel
Parts:
- removed JTAG1: (no value), microbuilder_v3:JTAG-CORTEXM3SMT
- removed L1: 2.2µH, SparkFun:INDUCTOR1007
- removed U$2: AA_HOLDER, fbri:AA_HOLDER
- removed U4: ADP1607ACPZN-R7, ADP1607:ADP1607ACPZN-R7
- added C20: 18pF, microbuilder_v3:CAP_CERAMIC_0402
- added C21, C22: 100nF, microbuilder_v3:CAP_CERAMIC_0402
- added D2: GREEN, led:LEDCHIPLED_0603
- added R3: 100kΩ, microbuilder_v3:RESISTOR_0402
- added R4, R5, R6: 10kΩ, microbuilder_v3:RESISTOR_0402
- added U$33: SE880, fbri:SE880
- added U$51: M04X2, fbri:M04X2
- added U$74: M05, fbri:M05
- added U$75: TG-5006CJ, fbri:TG-5006CJ
- added U3: SN74LVC1G32DCKR, SN74LVC1G32DCKR:SN74LVC1G32DCKR
- added Y1: ABS05, fbri:ABS05
- C18: value 10µF -> 100nF; device resistor:C-EUC0603K -> microbuilder_v3:CAP_CERAMIC_0402
- C19: value 10µF -> 18pF; device resistor:C-EUC0603K -> microbuilder_v3:CAP_CERAMIC_0402
- R1: value 100kΩ -> 10kΩ
- R2: value 240kΩ -> 100kΩ
Connections:
- net LED renamed LED1
- removed net !MR: JTAG1.10, U$19.!MR
- removed net FB: R1.1, R2.2, U4.FB
- removed net SW: L1.2, U4.SW
- new net EXT!RESET: R1.2, U$74.2, U3.A
- new net LED2: D2.C, U1.PA16
- new net N$2: U$33.VBB_I, U$33.VREG_O
- new net N$3: R6.2, U$33.GPIO0
- new net N$4: R4.1, U$33.CTS_SPI
- new net N$5: R5.2, U$33.GPIO1
- new net RTC_XI: C19.P$1, U$33.RTC_XI, Y1.1
- new net RTC_XO: C20.P$1, U$33.RTC_XO, Y1.2
- new net SAM_XOSC: C18.P$1, R2.2, R3.1, U1.PA14
- new net SE_ON_OFF: U$33.ON_OFF, U1.PA04
- new net WDI!RESET: U$19.!RESET, U3.B
- net !RESET: now also U$33.NSRESET, U$48.9_V_RESET, U3.Y; no longer U$19.!RESET
- net 1.2V: now also U$51.5; no longer C18.1, L1.1, U$2.+, U4.EN, U4.VIN
- net 1.8V: now also C21.P$1, D2.A, R3.2, R4.2, U$19.!MR, U$33.VDD, U$33.VKA, U$51.3, U$74.3, U3.VCC; no longer C19.1, JTAG1.1, R1.2, U4.VOUT
- net GIMO: now also U$33.RX
- net GND: now also C19.P$2, C20.P$2, C21.P$2, R1.1, R5.1, R6.1, U$33.GND1, U$33.GND10, U$33.GND2, U$33.GND3, U$33.GND4, U$33.GND5, U$33.GND6, U$33.GND7, U$33.GND8, U$33.GND9, U$51.1, U$51.2, U$74.1, U3.GND; no longer C18.2, C19.2, JTAG1.3, JTAG1.5, U$2.-, U4.EP, U4.GND
- net GOMI: now also U$33.TX
- net GPS_ANT: now also U$33.RF_IN
- net SI_SDN: now also U1.PA17; no longer U1.PA16
- net SWDCLK: now also U$74.5; no longer JTAG1.4
- net SWDIO: now also U$74.4; no longer JTAG1.2
- net TCXO_OUT: now also C18.P$2; no longer U1.PA17
- net TIMEPULSE: now also U$33.TM
Other:
- note added: "GND, GND, 1.8V, Vbattery, DATA"
- note added: "NC, GND, Status, Vsolar, CLK"
- note removed: "(GLCK_IO[3])"
- note removed: "ADP1607 Step-Up DC-DC Converter VBatt -> 1.8V"
- note removed: "Second +ve terminal is the 2nd physical connection on the holder"
- moved on the sheet: C1, C10, C11, C12, C13, C14, C15, C16, C17, C18, C19, C2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

Commit message: Routing on the bottom half of the main board almost done
Parts:
- added C23: 100nF, microbuilder_v3:CAP_CERAMIC_0402
- added R10: 22kΩ, microbuilder_v3:RESISTOR_0402
- added R7, R8, R9: 10kΩ, microbuilder_v3:RESISTOR_0402
Connections:
- new net I2C_CLK: R8.1, U$51.8, U1.PA05
- new net I2C_DATA: R7.1, U$51.7, U1.PA04
- new net SE_TCXO_CLK: U$33.TCXO_CLK, U$75.OUT
- new net SE_VCO_TCXO: C22.P$1, U$33.VCC_TCXO, U$75.VCC
- new net VBATT_SENSE: R10.1, R9.2, U1.PA11
- new net VSOLAR: U$51.6, U1.PA03
- net 1.2V: now also R10.2; no longer U1.PA11
- net 1.8V: now also C23.P$1, R7.2, R8.2
- net GND: now also C22.P$2, C23.P$2, R9.1, U$75.GND
- net SE_ON_OFF: no longer U1.PA04
- net TIMEPULSE: now also U1.PA02; no longer U1.PA05
Other:
- note added: "(EXTINT[n])"
- note added: "GND, 1.8V, Vbattery, DATA"
- note added: "GND, NC, Vsolar, CLK"
- note removed: "(TC0 WC[1])"
- note removed: "GND, GND, 1.8V, Vbattery, DATA"
- note removed: "NC, GND, Status, Vsolar, CLK"
- moved on the sheet: C1, C11, C12, C13, C17, C2, C21, C22, C3, C4, C5, C6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

Commit message: Updated main board to v0.98.0
Parts:
- removed D1: GREEN, led:LEDCHIPLED_0603
- added C24, C25, C26, C27, C28, C29: 100nF, microbuilder_v3:CAP_CERAMIC_0402
- added C30: 100pF, microbuilder_v3:CAP_CERAMIC_0402
- added FB3: (no value), microbuilder_v3:FERRITE_0402
- added L1: 100nH, microbuilder_v3:INDUCTOR_0402
- added R13, R14: 0Ω, microbuilder_v3:RESISTOR_0402
- added R15, R17: 10kΩ, microbuilder_v3:RESISTOR_0402
- added R16: 15kΩ, microbuilder_v3:RESISTOR_0402
- added U$55: SI5356, si5356:SI5356
- added U4: AD8354, fbri:AD8354
Connections:
- removed net I2C_CLK: R8.1, U$51.8, U1.PA05
- removed net I2C_DATA: R7.1, U$51.7, U1.PA04
- removed net LED1: D1.C, U1.PA15
- new net AMPL_OUT: C28.P$1, L1.1, U4.VOUT
- new net AMPL_VPOS: C29.P$1, C30.P$1, FB3.P$1, L1.2, U4.VPOS
- new net CLKIN: R14.1, U$55.CLKIN
- new net HF: C28.P$2
- new net HF_CLK: C27.P$1, U$55.CLK2
- new net INPT: C27.P$2, U4.INPT
- new net INTR: R17.1, U$55.INTR
- new net N$7: U$55.CLK7
- new net SCL: R8.1, U$51.8, U$55.SCL, U1.PA05
- new net SDA: R7.1, U$51.7, U$55.SDA, U1.PA04
- new net SSC_DIS: R15.1, R16.2, U$55.SSC_DIS
- new net XA: C26.P$2, U$55.XA
- new net XB: R13.1, U$55.XB
- net !RESET: now also U$51.4
- net 1.8V: now also C24.P$1, C25.P$1, FB3.P$2, R15.2, R17.2, U$55.VCC1, U$55.VCC2, U$55.VDDO_A, U$55.VDDO_B, U$55.VDDO_C, U$55.VDDO_D; no longer D1.A
- net GND: now also C24.P$2, C25.P$2, C29.P$2, C30.P$2, R13.2, R14.2, R16.1, U$55.!OE, U$55.GND, U$55.GND_PAD, U$55.I2C_LSB, U4.COM1, U4.COM1_, U4.COM2, U4.EPAD, U4._COM2
- net SE_ON_OFF: now also U1.PA15
- net TCXO_OUT: now also C26.P$1
Other:
- note added: "All VDDOs must be connected to a supply >1.5V"
- note added: "GND, !RESET!, Vsolar, CLK"
- note removed: "GND, NC, Vsolar, CLK"

Commit message: Actually update main board to v0.98.0
Parts:
- removed U$23: TG-5006CJ, fbri:TG-5006CJ
- removed U$48: UBLOX_MAX, Ava:UBLOX_MAX
- added U44: AD8354, fbri:AD8354
- added U8: SN74LVC1G32DCKR, SN74LVC1G32DCKR:SN74LVC1G32DCKR
- C17: value 2.2µF -> 100nF
- C19, C20: value 18pF -> 100nF
- C21: value 100nF -> 2.2µF
- C22, C23: value 100nF -> 18pF
- R10: value 22kΩ -> 100kΩ
- R2, R3: value 100kΩ -> 10kΩ
- R8: value 10kΩ -> 22kΩ
- R9: value 10kΩ -> 100kΩ
- U3: value SN74LVC1G32DCKR -> UBLOX_MAX; device SN74LVC1G32DCKR:SN74LVC1G32DCKR -> Ava:UBLOX_MAX
- U4: value AD8354 -> S25FS-S; device fbri:AD8354 -> fbri:S25FS-S
- U5: value S25FS-S -> TG-5006CJ; device fbri:S25FS-S -> fbri:TG-5006CJ
- renumbered U$19 to U7, U$33 to U9, U$75 to U6
Connections:
- net HF renamed HF_ANT
- net !RESET: now also U3.9_V_RESET, U8.Y; no longer U$48.9_V_RESET, U3.Y
- net 1.2V: now also R8.2; no longer R10.2
- net 1.8V: now also C17.P$1, C19.P$1, R10.2, R2.2, U3.7_VCC_IO, U3.8_VCC, U4.VDD, U8.VCC; no longer C21.P$1, C23.P$1, R7.2, R8.2, U$48.7_VCC_IO, U$48.8_VCC, U3.VCC, U5.VDD
- net AMPL_OUT: now also U44.VOUT; no longer U4.VOUT
- net AMPL_VPOS: now also U44.VPOS; no longer U4.VPOS
- net EXT!RESET: now also U8.A; no longer U3.A
- net GIMO: now also U3.3_RXD1; no longer U$48.3_RXD1
- net GND: now also R7.1, U3.10_GND, U3.12_GND, U3.1_GND, U4.GND_PAD, U4.VSS, U44.COM1, U44.COM1_, U44.COM2, U44.EPAD, U44._COM2, U5.GND, U8.GND; no longer R2.1, U$23.GND, U$48.10_GND, U$48.12_GND, U$48.1_GND, U3.GND, U4.COM1, U4.COM1_, U4.COM2, U4.EPAD, U4._COM2, U5.GND_PAD, U5.VSS
- net GOMI: now also U3.2_TXD1; no longer U$48.2_TXD1
- net GPS_ANT: now also U3.11_RF_IN; no longer U$48.11_RF_IN
- net INPT: now also U44.INPT; no longer U4.INPT
- net MEM_CSN: now also U4.CSN; no longer U5.CSN
- net MEM_MISO: now also U4.SO/IO1; no longer U5.SO/IO1
- net MEM_MOSI: now also U4.SI/IO0; no longer U5.SI/IO0
- net MEM_SCK: now also U4.SCK; no longer U5.SCK
- net MEM_WPN: now also U4.WPN/IO2; no longer U5.WPN/IO2
- net RADIO_VDD: now also C21.P$1; no longer C17.P$1
- net RTC_XI: now also C22.P$1; no longer C19.P$1
- net RTC_XO: now also C23.P$1; no longer C20.P$1
- net SAM_XOSC: now also R10.1, R9.2; no longer R2.2, R3.1
- net SCL: now also R2.1; no longer R8.1
- net SDA: now also R3.1; no longer R7.1
- net SE_VCO_TCXO: now also C20.P$1; no longer C22.P$1
- net TCXO_OUT: now also U5.OUT; no longer U$23.OUT
- net TCXO_VDD: now also U5.VCC; no longer U$23.VCC
- net TIMEPULSE: now also U3.4_TIMEPULSE; no longer U$48.4_TIMEPULSE
- net VBATT_SENSE: now also R7.2, R8.1; no longer R10.1, R9.2
- net WDI!RESET: now also U8.B; no longer U3.B
Other:
- moved on the sheet: C17, C19, C20, C21, C22, C23, R10, R2, R3, R7, R8, R9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
