File: hardware/main-solar-hf/bristol_longshot.sch (EAGLE design)
At the start: 72 parts, among them U1 SAM_D20E, U2 SI4060, U3 UBLOX_MAX, U4 S25FS-S, U44 AD8354, U5 TG-5006CJ, U6 TG-5006CJ, U7 TPS3123, U8 SN74LVC1G32DCKR, U9 SE880, Y1 ABS05

Commit message: Moved to single-board solar tracker. Parts lists out of date!
Parts:
- removed U$51: M04X2, fbri:M04X2
- added C31, C41: 10µF, resistor:C-EUC0603K
- added C32, C33, C40: 1nF, microbuilder_v3:CAP_CERAMIC_0402
- added C34, C35, C36, C37, C38, C39, C42: 4.7µF, microbuilder_v3:CAP_CERAMIC_0402
- added D3, D4: BAT760, BAT760:BAT760
- added L8, L9: 2.2µH, SparkFun:INDUCTOR1007
- added R11, R19: 10kΩ, microbuilder_v3:RESISTOR_0402
- added R12: 1kΩ, microbuilder_v3:RESISTOR_0402
- added R18: 2.2kΩ, microbuilder_v3:RESISTOR_0402
- added R21: DNP, microbuilder_v3:RESISTOR_0402
- added U$113: XAL6060, XAL6060:XAL6060
- added U$19: SST25WF040BT-40I/NP, fbri:SST25WF040BT-40I/NP
- added U10: TPS62243, TPS62243:TPS62243
- added U11: TPS3808, TPS3808:TPS3808
- added U12: 74LVC1G04GW, 74LVC1G04GW_inverter:74LVC1G04GW
- added U13: SPV1040, spv1040:SPV1040
- added U14: LT4054ES5-4.2, XYKlib:LT4054ES5-4.2
- R2: value 10kΩ -> 82kΩ
- R3: value 10kΩ -> 220kΩ
- U4: value S25FS-S -> TPS62243; device fbri:S25FS-S -> TPS62243:TPS62243
Connections:
- net N$2 renamed SE_VREG
- net N$4 renamed SE_MODE_PULL
- net TANK renamed RF_TANK
- removed net 1.2V: R8.2, U$51.5
- new net BATTERY: C36.P$1, C38.P$1, D3.A, R21.2, R8.2, U14.BAT, U4.VIN
- new net BATTERY_BUCK_SW: L8.1, U4.SW
- new net BATTERY_EN: R11.1, U12.Y, U4.EN
- new net CHG_CONTROL: R18.1, U1.PA03
- new net CHG_STATUS: U14.CHRG
- new net CT: U11.CT
- new net LX1: U$113.2, U13.LX
- new net MPP-SET: C33.P$2, R12.2, U13.MPP-SET
- new net MPPT-VOUT-TANK: C37.P$1, C39.P$1, C42.P$1, D4.A, R21.1, R3.2, U10.VIN, U11.SENSE, U13.ICTRL+, U13.ICTRL-, U13.VOUT, U14.VCC
- new net PROG: R18.2, U14.PROG
- new net SPV_VCTRL1: C32.P$1, R2.2, R3.1, U13.VCTRL
- new net SUPERVISOR_VCC: C40.P$1, D3.C, D4.C, R11.2, R19.2, U11.VDD, U12.VCC
- new net TANK_BUCK_SW: L9.1, U10.SW
- new net TANK_EN: R19.1, U10.EN, U11.!RESET, U12.A
- net !RESET: no longer U$51.4
- net 1.8V: now also C31.1, C41.1, L8.2, L9.2, U$19.VDD, U10.FB, U4.FB; no longer R2.2, R3.2, U$51.3, U4.VDD
- net GIMO: now also U1.PA06; no longer U1.PA00
- net GND: now also C31.2, C32.P$2, C33.P$1, C34.P$2, C35.P$2, C36.P$2, C37.P$2, C38.P$2, C39.P$2, C40.P$2, C41.2, C42.P$2, R2.1, U$19.GND_PAD, U$19.VSS, U10.GND, U10.GND2, U10.MODE, U11.GND, U11.GND2, U12.GND, U13.GND, U14.GND, U4.GND, U4.GND2, U4.MODE; no longer U$51.1, U$51.2, U4.GND_PAD, U4.VSS
- net GOMI: now also U1.PA07; no longer U1.PA01
- net MEM_CSN: now also U$19.CSN; no longer U4.CSN
- net MEM_MISO: now also U$19.SO/IO1, U1.PA11; no longer U1.PA09, U4.SO/IO1
- net MEM_MOSI: now also U$19.SI/IO0, U1.PA08; no longer U1.PA06, U4.SI/IO0
- net MEM_SCK: now also U$19.SCK, U1.PA09; no longer U1.PA07, U4.SCK
- net MEM_WPN: now also U$19.WPN/IO2; no longer U1.PA08, U4.WPN/IO2
- net SCL: now also U1.PA01; no longer R2.1, U$51.8, U1.PA05
- net SDA: now also U1.PA00; no longer R3.1, U$51.7, U1.PA04
- net TIMEPULSE: now also U1.PA05; no longer U1.PA02
- net VBATT_SENSE: now also U1.PA02; no longer U1.PA11
- net VSOLAR: now also C34.P$1, C35.P$1, R12.1, U$113.1, U1.PA04, U13.XSHUT; no longer U$51.6, U1.PA03
Other:
- note added: "!MR! has internal pull-up"
- note added: "(AIN[0])"
- note added: "(AIN[4])"
- note added: "(DO: PAD0, SCK: PAD1, DOPO: 0x0)"
- note added: "(EXTINT[5])"
- note added: "(SERCOM2)"
- note added: "(TX: PAD2, TXPO: 0x1)"
- note added: "Choose so total current through divider is 2µA - 20µA"
- note added: "Enable: Vil = 0.4V, Vih=1V"
- note added: "Ichg = 150V / Rchg"
- note added: "Ichg can be measured by Vprog"
- note added: "Input Voltage: 2 - 6V"
- note added: "Leaving Ct open sets the reset time (transition battery->solar) to 20ms"
- note added: "Not actually an SMA connector"
- note added: "Rchg = 2.2kΩ gives Ichg = 70mA"
- note added: "Recommended input cap is 1µF"
- note added: "Still quite unsure on inductor value.. but 2.2µH is worth trying, since it would be much better than the recommended 10µH. Will the boost then run in inefficient discontinous mode????"
- note added: "The ICTRL inputs are just pulled to Vout as we're not using constant-current regulation"
- note added: "Undervoltage Lockout: 1.85V typ"
- note added: "Undervoltage lockout for MPP-SET under 0.24V"
- note added: "Vout = 1.25(R1/R2 + 1)"
- note removed: "(AIN[19])"
- note removed: "(DO: PAD2, SCK: PAD3, DOPO: 0x1)"
- note removed: "(EXTINT[n])"
- note removed: "(SERCOM1)"
- note removed: "(TX: PAD0, TXPO: 0x0)"
- note removed: "GND, !RESET!, Vsolar, CLK"
- note removed: "GND, 1.8V, Vbattery, DATA"
- moved on the sheet: R2, R3
