File: hardware/low-power-solar/bristol_longshot.sch (EAGLE design)
At the start: 143 parts, among them Q1 NX2301P, Q2 NX2301P, Q3 BSS84, Q4 BSS84, Q5 PBSS4130, Q6 PD84001, U1 SAM_D20E, U10 TPS71533DCKR, U11 TPS73118DBVT, U12 LTC4070EMS8EPBF, U13 74LVC1G04GW, U14 SIT1552, U15 74LVC1G04GW, U16 SIT1552, U17 TPS71533DCKR, U18 74LVC1G04GW, U2 SI4461, U3 SE880, U4 SST25WF040BT-40I/NP, U5 TG-5006CJ, U6 ADP1614ACPZ-1.3-R7, U7 ADM6823WYRJZ, U8 SN74LVC1G32DCKR, U9 TPS62243

Commit message: [low-power-solar] complete IC section of partslist, board order
Parts:
- L1: value XFL4030-4.7µF -> XFL4030-4.7µH
- R29, R33: value 1kΩ -> 100kΩ
- R6: value 1MΩ -> 100kΩ
- U10: value TPS71533DCKR -> SIT1552; device TPS71533DCKR:TPS71533DCKR -> fbri:SIT1552
- U11: value TPS73118DBVT -> SIT1552; device TPS73118DVBT:TPS73118DBVT -> fbri:SIT1552
- U13: value 74LVC1G04GW -> ADP1614ACPZ-1.3-R7; device 74LVC1G04GW_inverter:74LVC1G04GW -> ADP1614:ADP1614ACPZ-1.3-R7
- U14: value SIT1552 -> TPS71533DCKR; device fbri:SIT1552 -> TPS71533DCKR:TPS71533DCKR
- U15: value 74LVC1G04GW -> TPS71533DCKR; device 74LVC1G04GW_inverter:74LVC1G04GW -> TPS71533DCKR:TPS71533DCKR
- U16: value SIT1552 -> 74LVC1G04GW; device fbri:SIT1552 -> 74LVC1G04GW_inverter:74LVC1G04GW
- U17: value TPS71533DCKR -> 74LVC1G04GW; device TPS71533DCKR:TPS71533DCKR -> 74LVC1G04GW_inverter:74LVC1G04GW
- U6: value ADP1614ACPZ-1.3-R7 -> TPS73118DBVT; device ADP1614:ADP1614ACPZ-1.3-R7 -> TPS73118DVBT:TPS73118DBVT
- renumbered U$23 to U20, U$80 to U19
Connections:
- net 1.8V: now also U10.VCC, U17.VCC, U18.VCC; no longer U13.VCC, U15.VCC, U16.VCC
- net 7.5V: now also U14.IN; no longer U10.IN
- net BOOST_COMP: now also U13.COMP; no longer U6.COMP
- net BOOST_CURRENTLIMIT: now also U13.CLRES; no longer U6.CLRES
- net BOOST_FB: now also U13.FB; no longer U6.FB
- net BOOST_SOFTSTART: now also U13.SS; no longer U6.SS
- net BOOST_SUPPLY: now also U13.EN, U13.VIN; no longer U6.EN, U6.VIN
- net BOOST_SW: now also U13.SW, U13.SW_2; no longer U6.SW, U6.SW_2
- net GND: now also U10.GND1, U11.GND1, U13.EP, U13.GND_2; no longer U14.GND1, U16.GND1, U6.EP, U6.GND_2
- net GPS_VDD_SWITCHED: now also U11.VCC; no longer U14.VCC
- net LF_CLOCK_OUT: now also U10.OUT; no longer U16.OUT
- net RADIO_VDD: now also U16.VCC; no longer U18.VCC
- net RF_SW_V2: now also U16.Y; no longer U18.Y
- net RF_TCXO_REG_EN: now also U6.EN; no longer U11.EN
- net SE800_LF_OUT: now also U11.OUT; no longer U14.OUT
- net SI_GPIO0: now also U16.A; no longer U18.A
- net SI_GPIO2: now also U17.A; no longer U13.A
- net SI_GPIO3: now also U18.A; no longer U15.A
- net SKY_V1_1: now also U17.Y; no longer U13.Y
- net SKY_V2_1: now also U18.Y; no longer U15.Y
- net TCXO_REG_IN: now also U6.IN; no longer U11.IN
- net TCXO_REG_NR: now also U6.NR/FB; no longer U11.NR/FB
- net TCXO_VDD: now also U6.OUT; no longer U11.OUT
- net V_BUS: now also U15.IN; no longer U17.IN
- net V_GG: now also U14.OUT; no longer U10.OUT
- net V_SKY: now also U15.OUT; no longer U17.OUT
Other:
- moved on the sheet: U15, U17, U18

Commit message: [low-power-solar] finish of partslist
Parts:
- C4, C48: value TBD -> DNP
- L12: value TBD -> 0Ω
Changed lines of the file:
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@@
 <part name="R28" library="microbuilder_v3" deviceset="RESISTOR" device="_0402" value="330Ω"/>
 <part name="U$115" library="microbuilder_v3" deviceset="GND" device=""/>
-<part name="L12" library="microbuilder_v3" deviceset="INDUCTOR" device="_0402" value="TBD"/>
-<part name="C4" library="microbuilder_v3" deviceset="CAP_CERAMIC" device="_0402" value="TBD"/>
-<part name="C48" library="microbuilder_v3" deviceset="CAP_CERAMIC" device="_0402" value="TBD"/>
+<part name="L12" library="microbuilder_v3" deviceset="INDUCTOR" device="_0402" value="0Ω"/>
+<part name="C4" library="microbuilder_v3" deviceset="CAP_CERAMIC" device="_0402" value="DNP"/>
+<part name="C48" library="microbuilder_v3" deviceset="CAP_CERAMIC" device="_0402" value="DNP"/>
 <part name="U$116" library="microbuilder_v3" deviceset="GND" device=""/>
 <part name="U$117" library="microbuilder_v3" deviceset="GND" device=""/>

Commit message: [low-power-solar] update to partslist on ordering
Parts:
- R20, R21: value (none) -> 22Ω
- renumbered FB4 to FB3
Changed lines of the file:
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@@
 <part name="U$110" library="microbuilder_v3" deviceset="GND" device=""/>
 <part name="U$111" library="microbuilder_v3" deviceset="1.8V" device=""/>
-<part name="R20" library="microbuilder_v3" deviceset="RESISTOR" device="_0603MP"/>
-<part name="R21" library="microbuilder_v3" deviceset="RESISTOR" device="_0603MP"/>
+<part name="R20" library="microbuilder_v3" deviceset="RESISTOR" device="_0603MP" value="22Ω"/>
+<part name="R21" library="microbuilder_v3" deviceset="RESISTOR" device="_0603MP" value="22Ω"/>
 <part name="C49" library="microbuilder_v3" deviceset="CAP_CERAMIC" device="_0402" value="100nF"/>
 <part name="U$112" library="microbuilder_v3" deviceset="GND" device=""/>
@@
 <part name="JP2" library="SparkFun" deviceset="M02" device="LOCK" value="SOLAR_TERMINAL"/>
 <part name="U$91" library="microbuilder_v3" deviceset="GND" device=""/>
-<part name="FB4" library="microbuilder_v3" deviceset="FERRITE" device="_0603"/>
+<part name="FB3" library="microbuilder_v3" deviceset="FERRITE" device="_0603"/>
 <part name="R31" library="microbuilder_v3" deviceset="RESISTOR" device="_0402" value="1kΩ"/>
 <part name="R32" library="microbuilder_v3" deviceset="RESISTOR" device="_0402" value="1kΩ"/>
@@
 <instance part="JP2" gate="G$1" x="96.52" y="17.78" rot="MR180"/>
 <instance part="U$91" gate="G$1" x="106.68" y="292.1"/>
-<instance part="FB4" gate="G$1" x="472.44" y="88.9" rot="R90"/>
+<instance part="FB3" gate="G$1" x="472.44" y="88.9" rot="R90"/>
 <instance part="R31" gate="G$1" x="1066.8" y="236.22" rot="R90"/>
 <instance part="R32" gate="G$1" x="1066.8" y="193.04" rot="R90"/>
@@
 <wire x1="472.44" y1="78.74" x2="472.44" y2="81.28" width="0.1524" layer="91"/>
 <junction x="472.44" y="81.28"/>
-<pinref part="FB4" gate="G$1" pin="P$1"/>
+<pinref part="FB3" gate="G$1" pin="P$1"/>
 </segment>
 </net>
@@
 <pinref part="U$70" gate="G$1" pin="1.8V"/>
 <wire x1="472.44" y1="96.52" x2="472.44" y2="91.44" width="0.1524" layer="91"/>
-<pinref part="FB4" gate="G$1" pin="P$2"/>
-</segment>
-<segment>
+<pinref part="FB3" gate="G$1" pin="P$2"/>
+</segment>
+<segment>

Commit message: [low-power-solar] add values for rx section
Parts:
- C5: value DNP -> 5.1pF
- C6: value DNP -> 2.7pF
- L6, L7: value DNP -> 56nH
- R29, R33: value 100kΩ -> 10kΩ
Changed lines of the file:
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@@
 <part name="C9" library="microbuilder_v3" deviceset="CAP_CERAMIC" device="_0402" value="100pF"/>
 <part name="U$3" library="microbuilder_v3" deviceset="GND" device=""/>
-<part name="L6" library="microbuilder_v3" deviceset="INDUCTOR" device="_0402" value="DNP"/>
-<part name="C5" library="microbuilder_v3" deviceset="CAP_CERAMIC" device="_0402" value="DNP"/>
+<part name="L6" library="microbuilder_v3" deviceset="INDUCTOR" device="_0402" value="56nH"/>
+<part name="C5" library="microbuilder_v3" deviceset="CAP_CERAMIC" device="_0402" value="5.1pF"/>
 <part name="U$45" library="microbuilder_v3" deviceset="GND" device=""/>
-<part name="L7" library="microbuilder_v3" deviceset="INDUCTOR" device="_0402" value="DNP"/>
-<part name="C6" library="microbuilder_v3" deviceset="CAP_CERAMIC" device="_0402" value="DNP"/>
+<part name="L7" library="microbuilder_v3" deviceset="INDUCTOR" device="_0402" value="56nH"/>
+<part name="C6" library="microbuilder_v3" deviceset="CAP_CERAMIC" device="_0402" value="2.7pF"/>
 <part name="C28" library="microbuilder_v3" deviceset="CAP_CERAMIC" device="_0402" value="2.2µF"/>
 <part name="U$18" library="microbuilder_v3" deviceset="GND" device=""/>
@@
 <part name="R10" library="microbuilder_v3" deviceset="RESISTOR" device="_0402" value="100kΩ"/>
 <part name="U$65" library="microbuilder_v3" deviceset="GND" device=""/>
-<part name="R29" library="microbuilder_v3" deviceset="RESISTOR" device="_0402" value="100kΩ"/>
+<part name="R29" library="microbuilder_v3" deviceset="RESISTOR" device="_0402" value="10kΩ"/>
 <part name="Q5" library="PBSS4130" deviceset="PBSS4130" device=""/>
 <part name="U$121" library="microbuilder_v3" deviceset="GND" device=""/>
-<part name="R33" library="microbuilder_v3" deviceset="RESISTOR" device="_0402" value="100kΩ"/>
+<part name="R33" library="microbuilder_v3" deviceset="RESISTOR" device="_0402" value="10kΩ"/>
 </parts>
 <sheets>
